Commit message: post demo

File: models/block/model_black.urdf (robot description, URDF)
Before this commit: robot block, 1 links, 0 joints
Links:
- link block: mass 2.0 -> 0.5

File: models/block/model_blue.urdf (robot description, URDF)
Before this commit: robot block, 1 links, 0 joints
Links:
- link block: mass 2.0 -> 0.5

File: models/block/model_green.urdf (robot description, URDF)
Before this commit: robot block, 1 links, 0 joints
Links:
- link block: mass 2.0 -> 0.5

File: models/block/model_grey.urdf (robot description, URDF)
Before this commit: robot block, 1 links, 0 joints
Links:
- link block: mass 2.0 -> 0.5

File: models/block/model_purple.urdf (robot description, URDF)
Before this commit: robot block, 1 links, 0 joints
Links:
- link block: mass 2.0 -> 0.5

File: models/block/model_red.urdf (robot description, URDF)
Before this commit: robot block, 1 links, 0 joints
Links:
- link block: mass 2.0 -> 0.5

File: models/block/model_white.urdf (robot description, URDF)
Before this commit: robot block, 1 links, 0 joints
Links:
- link block: mass 2.0 -> 0.5

File: models/block/model_yellow.urdf (robot description, URDF)
Before this commit: robot block, 1 links, 0 joints
Links:
- link block: mass 2.0 -> 0.5

Commit message: instruction fix

File: models/block/model_black.urdf (robot description, URDF)
Before this commit: robot block, 1 links, 0 joints
Links:
- link block: mass 0.5 -> 0.04

File: models/block/model_blue.urdf (robot description, URDF)
Before this commit: robot block, 1 links, 0 joints
Links:
- link block: mass 0.5 -> 0.04

File: models/block/model_green.urdf (robot description, URDF)
Before this commit: robot block, 1 links, 0 joints
Links:
- link block: mass 0.5 -> 0.04

File: models/block/model_grey.urdf (robot description, URDF)
Before this commit: robot block, 1 links, 0 joints
Links:
- link block: mass 0.5 -> 0.04

File: models/block/model_purple.urdf (robot description, URDF)
Before this commit: robot block, 1 links, 0 joints
Links:
- link block: mass 0.5 -> 0.04

File: models/block/model_red.urdf (robot description, URDF)
Before this commit: robot block, 1 links, 0 joints
Links:
- link block: mass 0.5 -> 0.04

File: models/block/model_white.urdf (robot description, URDF)
Before this commit: robot block, 1 links, 0 joints
Links:
- link block: mass 0.5 -> 0.04

File: models/block/model_yellow.urdf (robot description, URDF)
Before this commit: robot block, 1 links, 0 joints
Links:
- link block: mass 0.5 -> 0.04
